File: kicad/_autosave-kicad.kicad_pcb (KiCad board)
At the start: 2 copper layers, 68.8 x 53.6 mm, 9 parts, among them U1 74HC595, U2 74HC595, U3 AT28C256_40PIN_ZIF

Commit message: KiCad: Added schematic and PCB for Arduino Shield.
Other:
- board text added: "EEPROM Pin 1"
- board text added: "Erik van Zijst, 2019 erik.van.zijst@gmail.com https://github.com/erikvanzijst/eeprom"
- board text added: "v01"
Changed lines of the file:
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@@
   (general
     (thickness 1.6)
-    (drawings 10)
+    (drawings 18)
     (tracks 338)
     (zones 0)
@@
       (net 64 "Net-(XA1-PadMISO)"))
   )
+  (gr_text "Erik van Zijst, 2019\nerik.van.zijst@gmail.com\nhttps://github.com/erikvanzijst/eeprom" (at 191.008 105.41) (layer B.SilkS)
+    (effects (font (size 1 1) (thickness 0.15)) (justify left mirror))
+  )
+  (gr_text "EEPROM Pin 1" (at 185.166 66.294) (layer F.SilkS)
+    (effects (font (size 1 1) (thickness 0.15)))
+  )
+  (gr_line (start 191.77 67.056) (end 191.008 67.564) (layer F.SilkS) (width 0.12))
+  (gr_line (start 191.77 67.056) (end 191.008 66.548) (layer F.SilkS) (width 0.12))
+  (gr_line (start 191.77 67.056) (end 179.832 67.056) (layer F.SilkS) (width 0.12))
+  (gr_line (start 191.77 65.786) (end 191.77 68.202) (layer F.SilkS) (width 0.12))
+  (gr_text v01 (at 132.842 61.976) (layer B.Cu)
+    (effects (font (size 1.5 1.5) (thickness 0.3)) (justify mirror))
+  )
+  (gr_text v01 (at 133.096 61.976) (layer F.Cu)
+    (effects (font (size 1.5 1.5) (thickness 0.3)))
+  )
   (gr_text "EEPROM Programmer Shield for\nArduino UNO R3" (at 144.653 105.537) (layer F.SilkS)
